File: hardware/rpi-cm4-base-carrier/rpi-cm4-base-carrier.kicad_sch (KiCad schematic)
At the start: 0 parts

Commit message: Placed components
Other:
- title: Raspberry Pi Compute Module 4 Carrier Template -> Raspberry Pi Compute Module 4 Base Carrier
Changed lines of the file:
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@@
   (paper "A4")
   (title_block
-    (title "Raspberry Pi Compute Module 4 Carrier Template")
+    (title "Raspberry Pi Compute Module 4 Base Carrier")
     (date "2020-10-31")
     (rev "v01")
