File: hardware/rpi-cm4-base-carrier/rpi-cm4-base-carrier.kicad_pcb (KiCad board)
At the start: 2 copper layers, 40 x 55 mm, 1 part

Commit message: Finished schematic
Parts:
- added CR1: SMBJ5.0A-TR, footprints:SMBJ5.0A-TR, F.Cu at (87.9, 97.7)
- added D1: LED Green, LED_SMD:LED_0603_1608Metric, F.Cu at (93.9, 98.7)
- added D2: LED Red, LED_SMD:LED_0603_1608Metric, F.Cu at (69.7, 114.2)
- added J1: DNP, Connector_PinHeader_2.54mm:PinHeader_1x10_P2.54mm_Vertical, F.Cu at (135.0, 131.4)
- added J2: USB4105-GF-A, USB4105-GF-A:GCT_USB4105-GF-A, F.Cu at (164.0, 121.2)
- added J3: SM04B-SRSS-TB(LF)(SN), SM04B-SRSS-TB_LF__SN_:JST_SM04B-SRSS-TB(LF)(SN), F.Cu at (161.5, 88.5)
- added J4: USB_OTG, CM4IO:USB_Micro-B_EDAC_UCON00686, F.Cu at (128.1, 121.0)
- added JP1: SolderJumper_2_Open, Jumper:SolderJumper-2_P1.3mm_Open_RoundedPad1.0x1.5mm, F.Cu at (69.8, 111.1)
- added R1: 5.1k, Resistor_SMD:R_0603_1608Metric_Pad0.98x0.95mm_HandSolder, F.Cu at (65.2, 123.6)
- added R2: 1k, Resistor_SMD:R_0603_1608Metric_Pad0.98x0.95mm_HandSolder, F.Cu at (74.2, 105.6)
- added R3: DNP, Resistor_SMD:R_0603_1608Metric_Pad0.98x0.95mm_HandSolder, F.Cu at (69.8, 105.6)
- added R4: 5.1k, Resistor_SMD:R_0603_1608Metric_Pad0.98x0.95mm_HandSolder, F.Cu at (74.2, 108.8)
- added R5: DNP, Resistor_SMD:R_0603_1608Metric_Pad0.98x0.95mm_HandSolder, F.Cu at (94.0, 96.1)
- added R6: 1k, Resistor_SMD:R_0603_1608Metric_Pad0.98x0.95mm_HandSolder, F.Cu at (69.8, 108.1)
- added R7: 2.2K 1%, Resistor_SMD:R_0603_1608Metric_Pad0.98x0.95mm_HandSolder, F.Cu at (113.3, 98.6)
- added R8: 2.2K 1%, Resistor_SMD:R_0603_1608Metric_Pad0.98x0.95mm_HandSolder, F.Cu at (113.3, 96.1)
- added U1: 74LVC1G07SE-7, Package_TO_SOT_SMD:SOT-353_SC-70-5, F.Cu at (78.5, 106.3)
- added U2: TPD2EUSB30, Package_TO_SOT_SMD:Texas_DRT-3, F.Cu at (112.4, 101.1)
Connections:
- Module1 pad 1: Net-(Module1-Pad1) -> GND
- Module1 pad 101: Net-(Module1-Pad101) -> /CM4 High Speed/USB_OTG_ID
- Module1 pad 103: Net-(Module1-Pad103) -> /CM4 High Speed/USB2_N
- Module1 pad 105: Net-(Module1-Pad105) -> /CM4 High Speed/USB2_P
- Module1 pad 107: Net-(Module1-Pad107) -> GND
- Module1 pad 108: Net-(Module1-Pad108) -> GND
- Module1 pad 113: Net-(Module1-Pad113) -> GND
- Module1 pad 114: Net-(Module1-Pad114) -> GND
- Module1 pad 119: Net-(Module1-Pad119) -> GND
- Module1 pad 120: Net-(Module1-Pad120) -> GND
- Module1 pad 125: Net-(Module1-Pad125) -> GND
- Module1 pad 126: Net-(Module1-Pad126) -> GND
- Module1 pad 13: Net-(Module1-Pad13) -> GND
- Module1 pad 131: Net-(Module1-Pad131) -> GND
- Module1 pad 132: Net-(Module1-Pad132) -> GND
- Module1 pad 137: Net-(Module1-Pad137) -> GND
- Module1 pad 138: Net-(Module1-Pad138) -> GND
- Module1 pad 14: Net-(Module1-Pad14) -> GND
- Module1 pad 144: Net-(Module1-Pad144) -> GND
- Module1 pad 150: Net-(Module1-Pad150) -> GND
- Module1 pad 155: Net-(Module1-Pad155) -> GND
- Module1 pad 156: Net-(Module1-Pad156) -> GND
- Module1 pad 161: Net-(Module1-Pad161) -> GND
- Module1 pad 162: Net-(Module1-Pad162) -> GND
- Module1 pad 167: Net-(Module1-Pad167) -> GND
- Module1 pad 168: Net-(Module1-Pad168) -> GND
- Module1 pad 173: Net-(Module1-Pad173) -> GND
- Module1 pad 174: Net-(Module1-Pad174) -> GND
- Module1 pad 179: Net-(Module1-Pad179) -> GND
- Module1 pad 180: Net-(Module1-Pad180) -> GND
- Module1 pad 185: Net-(Module1-Pad185) -> GND
- Module1 pad 186: Net-(Module1-Pad186) -> GND
- Module1 pad 191: Net-(Module1-Pad191) -> GND
- Module1 pad 192: Net-(Module1-Pad192) -> GND
- Module1 pad 197: Net-(Module1-Pad197) -> GND
- Module1 pad 198: Net-(Module1-Pad198) -> GND
- Module1 pad 2: Net-(Module1-Pad2) -> GND
- Module1 pad 20: Net-(Module1-Pad20) -> /CM4 GPIO/EEPROM_nWP
- Module1 pad 21: Net-(Module1-Pad21) -> /CM4 GPIO/nLED_Activity
- Module1 pad 22: Net-(Module1-Pad22) -> GND
- Module1 pad 23: Net-(Module1-Pad23) -> GND
- Module1 pad 32: Net-(Module1-Pad32) -> GND
- Module1 pad 33: Net-(Module1-Pad33) -> GND
- Module1 pad 37: Net-(Module1-Pad37) -> /CM4 GPIO/GPIO7
- Module1 pad 38: Net-(Module1-Pad38) -> /CM4 GPIO/GPIO11
- Module1 pad 39: Net-(Module1-Pad39) -> /CM4 GPIO/GPIO8
- Module1 pad 40: Net-(Module1-Pad40) -> /CM4 GPIO/GPIO9
- Module1 pad 42: Net-(Module1-Pad42) -> GND
- Module1 pad 43: Net-(Module1-Pad43) -> GND
- Module1 pad 44: Net-(Module1-Pad44) -> /CM4 GPIO/GPIO10
- Module1 pad 51: Net-(Module1-Pad51) -> /CM4 GPIO/GPIO15
- Module1 pad 52: Net-(Module1-Pad52) -> GND
- Module1 pad 53: Net-(Module1-Pad53) -> GND
- Module1 pad 55: Net-(Module1-Pad55) -> /CM4 GPIO/GPIO14
- Module1 pad 58: Net-(Module1-Pad58) -> /CM4 GPIO/GPIO2
- Module1 pad 59: Net-(Module1-Pad59) -> GND
- Module1 pad 60: Net-(Module1-Pad60) -> GND
- Module1 pad 65: Net-(Module1-Pad65) -> GND
- Module1 pad 66: Net-(Module1-Pad66) -> GND
- Module1 pad 7: Net-(Module1-Pad7) -> GND
- Module1 pad 71: Net-(Module1-Pad71) -> GND
- Module1 pad 74: Net-(Module1-Pad74) -> GND
- Module1 pad 77: Net-(Module1-Pad77) -> +5V
- Module1 pad 78: Net-(Module1-Pad78) -> +3.3V
- Module1 pad 79: Net-(Module1-Pad79) -> +5V
- Module1 pad 8: Net-(Module1-Pad8) -> GND
- Module1 pad 81: Net-(Module1-Pad81) -> +5V
- Module1 pad 83: Net-(Module1-Pad83) -> +5V
- Module1 pad 84: Net-(Module1-Pad84) -> +3.3V
- Module1 pad 85: Net-(Module1-Pad85) -> +5V
- Module1 pad 86: Net-(Module1-Pad86) -> +3.3V
- Module1 pad 87: Net-(Module1-Pad87) -> +5V
- Module1 pad 88: Net-(Module1-Pad88) -> +1.8V
- Module1 pad 90: Net-(Module1-Pad90) -> +1.8V
- Module1 pad 93: Net-(Module1-Pad93) -> /CM4 GPIO/nRPIBOOT
- Module1 pad 95: Net-(Module1-Pad95) -> /CM4 GPIO/nPWR_LED
- Module1 pad 98: Net-(Module1-Pad98) -> GND

Commit message: Placed components
Parts:
- JP1: moved to B.Cu
- moved R1 105.8 mm to (170.0, 109.0), turned to 180 degrees
- moved R3 100.6 mm to (170.0, 96.0)
- moved JP1 100.2 mm to (170.0, 115.0)
- moved R4 95.9 mm to (170.0, 106.0), turned to 180 degrees
- moved CR1 84.0 mm to (170.0, 115.0), turned to 90 degrees
- moved R5 76.0 mm to (170.0, 93.0)
- moved R6 56.2 mm to (123.0, 90.0), turned to -90 degrees
- moved D2 55.8 mm to (120.0, 90.0), turned to -90 degrees
- moved J1 55.5 mm to (174.5, 92.5), turned to 0 degrees
- moved R2 52.6 mm to (123.0, 86.0), turned to -90 degrees
- moved U1 45.2 mm to (122.0, 94.0), turned to 90 degrees
- moved D1 29.0 mm to (120.0, 86.0), turned to -90 degrees
- moved U2 21.9 mm to (124.0, 119.7), turned to 90 degrees
- moved R7 11.4 mm to (122.0, 106.0), turned to 180 degrees
- moved R8 11.1 mm to (122.0, 103.0)
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Connections:
- J3 pad 4: GND -> /CM4 GPIO/GPIO3
- Module1 pad 56: Net-(Module1-Pad56) -> /CM4 GPIO/GPIO3
- R5 pad 2: GND -> /CM4 GPIO/GPIO3
Other:
- board size 40 x 55 mm -> 60 x 55 mm

Commit message: Pretended to route USB lines
Parts:
- turned R7 to 0 degrees
- turned R8 to 180 degrees
Routing:
- net /CM4 High Speed/USB2_P: track 0.00 -> 21.9 mm
- net /CM4 High Speed/USB2_N: track 0.00 -> 18.7 mm
- net GND: track 0.00 -> 0.62 mm, vias 0 -> 1
Changed lines of the file:
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@@
   )
   (module "Resistor_SMD:R_0603_1608Metric_Pad0.98x0.95mm_HandSolder" (layer "F.Cu")
-    (at 122 106 180)
+    (at 122 106)
     (descr "Resistor SMD 0603 (1608 Metric), square (rectangular) end terminal, IPC_7351 nominal with elongated pad for handsoldering. (Body size source: IPC-SM-782 page 72, https://www.pcb-3d.com/wordpress/wp-content/uploads/ipc-sm-782a_amendment_1_and_2.pdf), generated with kicad-footprint-generator")
     (tags "resistor handsolder")
@@
     (fp_line (start 0.8 0.4125) (end -0.8 0.4125) (layer "F.Fab") (width 0.1))
     (fp_line (start -0.8 0.4125) (end -0.8 -0.4125) (layer "F.Fab") (width 0.1))
-    (pad "1" smd roundrect (at -0.9125 0 180) (size 0.975 0.95) (layers "F.Cu" "F.Paste" "F.Mask") (roundrect_rratio 0.25)
+    (pad "1" smd roundrect (at -0.9125 0) (size 0.975 0.95) (layers "F.Cu" "F.Paste" "F.Mask") (roundrect_rratio 0.25)
       (net 87 "Net-(J4-Pad1)"))
-    (pad "2" smd roundrect (at 0.9125 0 180) (size 0.975 0.95) (layers "F.Cu" "F.Paste" "F.Mask") (roundrect_rratio 0.25)
+    (pad "2" smd roundrect (at 0.9125 0) (size 0.975 0.95) (layers "F.Cu" "F.Paste" "F.Mask") (roundrect_rratio 0.25)
       (net 98 "/CM4 High Speed/USB_OTG_ID"))
     (model "${KISYS3DMOD}/Resistor_SMD.3dshapes/R_0603_1608Metric.wrl"
@@
   )
   (module "Resistor_SMD:R_0603_1608Metric_Pad0.98x0.95mm_HandSolder" (layer "F.Cu")
-    (at 122 103)
+    (at 122 103 180)
     (descr "Resistor SMD 0603 (1608 Metric), square (rectangular) end terminal, IPC_7351 nominal with elongated pad for handsoldering. (Body size source: IPC-SM-782 page 72, https://www.pcb-3d.com/wordpress/wp-content/uploads/ipc-sm-782a_amendment_1_and_2.pdf), generated with kicad-footprint-generator")
     (tags "resistor handsolder")
@@
     (fp_line (start 0.8 0.4125) (end -0.8 0.4125) (layer "F.Fab") (width 0.1))
     (fp_line (start -0.8 0.4125) (end -0.8 -0.4125) (layer "F.Fab") (width 0.1))
-    (pad "1" smd roundrect (at -0.9125 0) (size 0.975 0.95) (layers "F.Cu" "F.Paste" "F.Mask") (roundrect_rratio 0.25)
+    (pad "1" smd roundrect (at -0.9125 0 180) (size 0.975 0.95) (layers "F.Cu" "F.Paste" "F.Mask") (roundrect_rratio 0.25)
       (net 98 "/CM4 High Speed/USB_OTG_ID"))
-    (pad "2" smd roundrect (at 0.9125 0) (size 0.975 0.95) (layers "F.Cu" "F.Paste" "F.Mask") (roundrect_rratio 0.25)
+    (pad "2" smd roundrect (at 0.9125 0 180) (size 0.975 0.95) (layers "F.Cu" "F.Paste" "F.Mask") (roundrect_rratio 0.25)
       (net 3 "GND"))
     (model "${KISYS3DMOD}/Resistor_SMD.3dshapes/R_0603_1608Metric.wrl"
@@
     (style (thickness 0.15) (arrow_length 1.27) (text_position_mode 0) (extension_height 0.58642) (extension_offset 0.5) keep_text_aligned)
   )
+  (segment (start 123.575 119.7) (end 122.95 119.7) (width 0.2) (layer "F.Cu") (net 3))
+  (via (at 122.95 119.7) (size 0.508) (drill 0.254) (layers "F.Cu" "B.Cu") (net 3))
+  (segment (start 129.881894 120.1562) (end 125.582503 120.1562) (width 0.75) (layer "F.Cu") (net 81))
+  (segment (start 123.745999 120.254001) (end 122.704001 120.254001) (width 0.2) (layer "F.Cu") (net 81))
+  (segment (start 134.3512 115.686894) (end 129.881894 120.1562) (width 0.75) (layer "F.Cu") (net 81))
+  (segment (start 132.838094 112) (end 134.3512 113.513106) (width 0.75) (layer "F.Cu") (net 81))
+  (segment (start 123.95 120.05) (end 123.745999 120.254001) (width 0.2) (layer "F.Cu") (net 81))
+  (segment (start 132.2 112) (end 132.838094 112) (width 0.75) (layer "F.Cu") (net 81))
+  (segment (start 124.425 120.05) (end 123.95 120.05) (width 0.2) (layer "F.Cu") (net 81))
+  (segment (start 124.425 120.05) (end 125.476303 120.05) (width 0.2) (layer "F.Cu") (net 81))
+  (segment (start 131.7 112.5) (end 132 112.2) (width 0.2) (layer "F.Cu") (net 81))
+  (segment (start 122.45 120) (end 120.82 120) (width 0.2) (layer "F.Cu") (net 81))
+  (segment (start 134.3512 113.513106) (end 134.3512 115.686894) (width 0.75) (layer "F.Cu") (net 81))
+  (segment (start 125.476303 120.05) (end 125.582503 120.1562) (width 0.2) (layer "F.Cu") (net 81))
+  (segment (start 122.704001 120.254001) (end 122.45 120) (width 0.2) (layer "F.Cu") (net 81))
+  (segment (start 131.08 112.5) (end 131.7 112.5) (width 0.2) (layer "F.Cu") (net 81))
+  (segment (start 132 112.2) (end 132.2 112) (width 0.2) (layer "F.Cu") (net 81))
+  (segment (start 122.704001 119.145999) (end 122.5 119.35) (width 0.2) (layer "F.Cu") (net 82))
+  (segment (start 123.95 119.35) (end 123.745999 119.145999) (width 0.2) (layer "F.Cu") (net 82))
+  (segment (start 131.08 112.9) (end 131.7 112.9) (width 0.2) (layer "F.Cu") (net 82))
+  (segment (start 133.4488 115.313106) (end 129.508106 119.2538) (width 0.75) (layer "F.Cu") (net 82))
+  (segment (start 125.486303 119.35) (end 125.582503 119.2538) (width 0.2) (layer "F.Cu") (net 82))
+  (segment (start 122.5 119.35) (end 120.82 119.35) (width 0.2) (layer "F.Cu") (net 82))
+  (segment (start 132.2 113.4) (end 132.961906 113.4) (width 0.75) (layer "F.Cu") (net 82))
+  (segment (start 124.425 119.35) (end 125.486303 119.35) (width 0.2) (layer "F.Cu") (net 82))
+  (segment (start 124.425 119.35) (end 123.95 119.35) (width 0.2) (layer "F.Cu") (net 82))
+  (segment (start 132 113.2) (end 132.2 113.4) (width 0.2) (layer "F.Cu") (net 82))
+  (segment (start 132.961906 113.4) (end 133.4488 113.886894) (width 0.75) (layer "F.Cu") (net 82))
+  (segment (start 131.7 112.9) (end 132 113.2) (width 0.2) (layer "F.Cu") (net 82))
+  (segment (start 123.745999 119.145999) (end 122.704001 119.145999) (width 0.2) (layer "F.Cu") (net 82))
+  (segment (start 133.4488 113.886894) (end 133.4488 115.313106) (width 0.75) (layer "F.Cu") (net 82))
+  (segment (start 129.508106 119.2538) (end 125.582503 119.2538) (width 0.75) (layer "F.Cu") (net 82))
   (zone (net 0) (net_name "") (layers F&B.Cu) (name "Wireless Keepout") (hatch edge 0.508)
     (connect_pads (clearance 0))

Commit message: Finished with PCB layout
Parts:
- added REF**: Fiducial_1mm_Mask2mm, Fiducial:Fiducial_1mm_Mask2mm, F.Cu at (120.0, 131.5)
- added REF**: Fiducial_1mm_Mask2mm, Fiducial:Fiducial_1mm_Mask2mm, F.Cu at (173.0, 80.5)
- moved R3 4.00 mm to (170.1, 92.0)
- moved R1 4.00 mm to (170.0, 105.0)
- moved R5 2.00 mm to (170.1, 95.0)
- moved R4 2.00 mm to (170.0, 108.0)
- moved J3 0.50 mm to (171.0, 85.5)
- moved J4 0.10 mm to (118.1, 120.0)
- turned JP1 to -90 degrees
Routing:
- net +3.3V: track 0.00 -> 89.7 mm
- net /CM4 GPIO/nLED_Activity: track 0.00 -> 52.0 mm, vias 0 -> 2
- net /CM4 GPIO/nPWR_LED: track 0.00 -> 47.3 mm, vias 0 -> 2
- net +5V: track 0.00 -> 46.9 mm
- net /CM4 GPIO/nRPIBOOT: track 0.00 -> 32.4 mm, vias 0 -> 1
- net /CM4 GPIO/GPIO3: track 0.00 -> 30.7 mm, vias 0 -> 2
- net /CM4 GPIO/GPIO2: track 0.00 -> 28.2 mm, vias 0 -> 2
- net Net-(J2-PadA5): track 0.00 -> 24.2 mm
- net /CM4 High Speed/USB_OTG_ID: track 0.00 -> 18.3 mm
- net Net-(J2-PadB5): track 0.00 -> 17.4 mm
- net /CM4 GPIO/GPIO7: track 0.00 -> 16.6 mm, vias 0 -> 1
- net /CM4 GPIO/GPIO8: track 0.00 -> 15.5 mm, vias 0 -> 1
- net Net-(J4-Pad1): track 0.00 -> 15.3 mm
- net /CM4 GPIO/GPIO14: track 0.00 -> 13.7 mm, vias 0 -> 1
- net /CM4 GPIO/GPIO10: track 0.00 -> 13.5 mm, vias 0 -> 1
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- added copper zone on B.Cu, net GND
- added copper zone on F.Cu, net GND
Other:
- board text added: "RPi CM4 Base Carrier"
- board text removed: "RPi CM4 Carrier Template"
